Commit message: Nav: Regulated Pure Pursuit, wider inflation, skid-steer effective track factor

File: ros2_ws/src/shopping_robot_description/urdf/shopping_robot.urdf.xacro (robot description, xacro)
@@ -5,4 +5,5 @@
   <xacro:property name="height" value="0.18"/>
   <xacro:property name="wheel_radius" value="0.10"/>
+  <xacro:property name="skid_track_factor" value="2.0"/>
   <xacro:property name="wheel_width" value="0.04"/>
   <xacro:arg name="anchor_count" default="3"/>
@@ -48,5 +49,7 @@
     <plugin filename="libignition-gazebo-diff-drive-system.so" name="ignition::gazebo::systems::DiffDrive">
       <left_joint>front_left_joint</left_joint><left_joint>rear_left_joint</left_joint><right_joint>front_right_joint</right_joint><right_joint>rear_right_joint</right_joint>
-      <wheel_separation>${width-wheel_width}</wheel_separation><wheel_radius>${wheel_radius}</wheel_radius>
+      <!-- Effective track for skid steer: lateral wheel scrub resists yaw, so the geometric track (~0.44 m)
+         barely turns the base at small angular commands. skid_track_factor scales it (calibrate on the real base). -->
+      <wheel_separation>${(width-wheel_width)*skid_track_factor}</wheel_separation><wheel_radius>${wheel_radius}</wheel_radius>
       <topic>cmd_vel</topic><odom_topic>wheel_odom</odom_topic><tf_topic>wheel_tf</tf_topic><frame_id>odom</frame_id><child_frame_id>base_footprint</child_frame_id><odom_publish_frequency>50</odom_publish_frequency>
       <max_linear_velocity>0.6</max_linear_velocity><max_angular_velocity>1.2</max_angular_velocity>
